File: PCB/cncvac.kicad_pcb (KiCad board)
At the start: 4 copper layers, 48.9 x 59.7 mm, 34 parts, among them J1 AVR-ISP-6, J2 24VAC, SW1 SW_SPST, U1 ATtiny841-SS, U2 MICRF112YMM, U3 LTV-357T, Y1 13.56MHz, Y2 8MHz

Commit message: givver
Parts:
- added JP1: 5V, Jumper:SolderJumper-2_P1.3mm_Open_RoundedPad1.0x1.5mm, F.Cu at (46.5, 69.1)
- added R5: 1k, Resistor_SMD:R_0402_1005Metric, F.Cu at (43.0, 70.1)
- J2: value 24VAC -> TRIG
- moved J1 1.01 mm to (64.4, 92.3)
- moved BT1 0.31 mm to (77.8, 83.0)
Routing:
- net VDD: track 83.7 -> 73.6 mm
- net /TRIG+: track 4.47 -> 13.7 mm, vias 0 -> 2
- net Net-(JP1-A): track 0.00 -> 4.04 mm
- net /ASK: track 12.6 -> 13.7 mm
- net /RST: track 21.8 -> 20.8 mm
- net /MISO: track 20.1 -> 19.1 mm
- net /SCK: track 24.8 -> 23.8 mm
- net /MOSI: track 14.6 -> 13.6 mm
Other:
- board text added: "Solder JP1 bridge to reduce trigger resistor from 1K to 500Ω (Better for 5V input)"
